File: PCB/GO-button/GO-button-QFN44.kicad_pcb (KiCad board)
At the start: 2 copper layers, 52 x 74 mm, 38 parts, among them J1 GT-USB-7010ASV, J2 AVR-ISP-6, SW1 SW_Push, SW2 SW_Push, SW3 SW_Push, SW4 SW_Push, SW5 SW_Push, SW6 TS-1187A-B-A-B, U1 ATmega32U4-A, Y1 X322516MLB4SI

Commit message: PCB REV 1.0.1
Parts:
- added C10: 0.1uF, Capacitor_SMD:C_0402_1005Metric, F.Cu at (116.7, 80.2)
- added C11: 0.1uF, Capacitor_SMD:C_0402_1005Metric, F.Cu at (139.2, 79.8)
- added C12: 0.1uF, Capacitor_SMD:C_0402_1005Metric, F.Cu at (115.3, 103.8)
- added C13: 0.1uF, Capacitor_SMD:C_0402_1005Metric, F.Cu at (135.7, 103.8)
- added C14: 0.1uF, Capacitor_SMD:C_0402_1005Metric, F.Cu at (129.3, 127.8)
- added R10: 4k7, Resistor_SMD:R_0402_1005Metric, F.Cu at (129.2, 112.2)
- added R11: 220E, Resistor_SMD:R_0402_1005Metric, F.Cu at (115.7, 80.2)
- added R6: 4k7, Resistor_SMD:R_0402_1005Metric, F.Cu at (118.2, 79.8)
- added R7: 4k7, Resistor_SMD:R_0402_1005Metric, F.Cu at (137.2, 79.8)
- added R8: 4k7, Resistor_SMD:R_0402_1005Metric, F.Cu at (124.2, 91.4)
- added R9: 4k7, Resistor_SMD:R_0402_1005Metric, F.Cu at (133.5, 92.2)
Connections:
- D1 pad 4: /MOSI -> Net-(D1-DIN)
- J2 pad 1: /MOSI -> /MISO
- J2 pad 4: /MISO -> /MOSI
- U1 pad 45: GND -> (no net)
Routing:
- net +5V: track 161.2 -> 173.6 mm, vias 6 -> 7
- net /MISO: track 25.6 -> 17.2 mm
- net /MOSI: track 23.3 -> 28.3 mm
- net Net-(D1-DIN): track 0.00 -> 3.78 mm
- net /SW5: track 29.4 -> 32.9 mm
- net /SW4: track 15.5 -> 16.8 mm
- net /SW3: track 9.88 -> 10.8 mm
- net GND: vias 18 -> 19
Other:
- board text added: "Jun. 2023"
- board text added: "Rev 1.0.1"
- board text removed: "Mar. 2023"
- board text removed: "Rev 1.0.0"
